Commit message: Avance proyecto [EDU]

File: proyecto/src/robot_description/urdf/robotRRR.urdf (robot description, URDF)
Before this commit: robot robot_rrr, 4 links, 3 joints
Links:
- added link end_effector_link; visual sphere radius=0.03
- link arm_link: geometry visual box size=0.05 0.05 0.30
Joints:
- added joint end_effector_joint: type fixed, parent forearm_link, child end_effector_link, origin xyz=0 0 0.45 rpy=0 0 0
- joint arm_joint: origin xyz=0 0 0.15 -> xyz=0 0 0.15 rpy=0 0 0
- joint forearm_joint: origin xyz=0 0 0.3 -> xyz=0 0 0.30 rpy=0 0 0
- joint shoulder_joint: origin xyz=0 0 0 -> xyz=0 0 0 rpy=0 0 0
